File: LED_driver.kicad_sch (KiCad schematic)
At the start: 14 parts, among them J4 LED_STRIP_CONNECTOR, Q3 UMW30N06, Q4 UMW30N06, Q5 UMW30N06, U6 MCP1416, U7 MCP1416, U8 MCP1416

Commit message: initial rev of design
Parts:
- removed J?: Screw_Terminal_01x03, symbol Connector:Screw_Terminal_01x03
- removed J?: Conn_01x03, symbol Connector_Generic:Conn_01x03
- added JP3: NEOPIXEL, Jumper:SolderJumper-2_P1.3mm_Open_RoundedPad1.0x1.5mm, symbol Jumper:SolderJumper_2_Open
- added JP4: Jumper_2_Bridged, Connector_PinHeader_2.54mm:PinHeader_1x02_P2.54mm_Vertical, symbol Jumper:Jumper_2_Bridged
- added R14, R15, R16: 100, Resistor_SMD:R_0805_2012Metric_Pad1.20x1.40mm_HandSolder, symbol Device:R_US
- C12, C13, C14: LCSC (none) -> C15850
- J4: value LED_STRIP_CONNECTOR -> LED 5050
- J7: renamed from J?; value Conn_01x03_Female -> NEOPIXEL; footprint (none) -> Connector_PinHeader_2.54mm:PinHeader_1x03_P2.54mm_Vertical; now left out of the parts list
Connections:
- net Earth: now also J7.1 (Pin_1)
- net V_{LED}: no longer C12.1, C13.1, C14.1, U6.2 (Vdd), U7.2 (Vdd), U8.2 (Vdd)
- net at U7.5 (OUT): now also R15.1; no longer Q4.1 (G)
- net at U6.5 (OUT): now also R14.1; no longer Q3.1 (G)
- net at Q5.1 (G): now also JP3.1 (A), JP4.1 (A), R16.2; no longer U8.5 (OUT)
- net Din: now reaches J7.2 (Pin_2)
- net Din: now also JP3.2 (B), JP4.2 (B)
- net V_{LED5V}: now reaches J7.3 (Pin_3)
- net V_{LED5V}: now also C12.1, C13.1, C14.1, U6.2 (Vdd), U7.2 (Vdd), U8.2 (Vdd)
- new net: Q4.1 (G), R15.2
- new net: Q3.1 (G), R14.2
- new net: R16.1, U8.5 (OUT)
Other:
- moved on the sheet: C12, C13, C14, D2, J4, J7, Q3, Q4, Q5, U6, U7, U8

Commit message: updated text, finalizing of board design, updated schematic rev number
Connections:
- net Earth: now also J7.3 (Pin_3); no longer J7.1 (Pin_1)
- net V_{LED5V}: now also J7.1 (Pin_1); no longer J7.3 (Pin_3)

Commit message: library changes, fixed model for dc jack
Other:
- title: IoT LED Strip Driver -> Spotify Reactive IoT LED Strip Driver
Changed lines of the file:
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@@
   (paper "A4")
   (title_block
-    (title "IoT LED Strip Driver")
+    (title "Spotify Reactive IoT LED Strip Driver")
     (date "2023-08-13")
-    (rev "v1.0")
+    (rev "v1.8-a")
     (comment 1 "A modular, internet connected LED strip driver")
+    (comment 2 "that reacts to the currently playing song on spotify")
   )
   (junction (at 92.075 97.155) (diameter 0) (color 0 0 0 0)
