File: USB_to_Serial.kicad_sch (KiCad schematic)
At the start: 15 parts, among them Q1 S8050_C105433, Q2 S8050_C105433, U1 CH340G, Y1 Crystal_12MHz

Commit message: initial rev of design
Parts:
- C1: LCSC (none) -> C49678
- C2, C3: LCSC (none) -> C1804
- Q1, Q2: footprint footprint:SOT-23-3_L2.9-W1.6-P1.90-LS2.8-BR -> Package_TO_SOT_SMD:SOT-23-3
- R1, R2: LCSC (none) -> C17414
- R8, R9: LCSC (none) -> C17710
- TP1, TP2, TP3, TP4: footprint TestPoint:TestPoint_Pad_D2.0mm -> TestPoint:TestPoint_Pad_D1.5mm
- U1: LCSC (none) -> C14267
- Y1: LCSC (none) -> C9002
Connections:
- net TXD: now reaches R8.1, U1.2 (TXD)
- net RXD: now reaches R9.1, U1.3 (RXD)
Changed lines of the file:
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@@
     (date "2023-05-03")
     (rev "v0.9")
-    (comment 1 "The hardware that leds the ESP8266 act as a USB device")
+    (comment 1 "A modular, internet connected LED strip driver")
   )
   (junction (at 236.22 69.85) (diameter 0) (color 0 0 0 0)
@@
     (effects (font (size 1.27 1.27)) (justify left bottom))
   )
+  (label "RXD" (at 140.335 71.12 0)
+    (effects (font (size 1.27 1.27)) (justify left bottom))
+  )
   (label "RTS" (at 144.78 88.9 0)
     (effects (font (size 1.27 1.27)) (justify left bottom))
@@
   )
   (label "RTS" (at 240.03 86.36 0)
+    (effects (font (size 1.27 1.27)) (justify left bottom))
+  )
+  (label "TXD" (at 140.335 68.58 0)
     (effects (font (size 1.27 1.27)) (justify left bottom))
   )
@@
       (effects (font (size 1.27 1.27)) (justify left))
     )
-    (property "Footprint" "footprint:SOT-23-3_L2.9-W1.6-P1.90-LS2.8-BR" (id 2) (at 223.52 76.2 0)
+    (property "Footprint" "Package_TO_SOT_SMD:SOT-23-3" (id 2) (at 223.52 76.2 0)
       (effects (font (size 1.27 1.27) italic) hide)
     )
@@
       (effects (font (size 1.27 1.27)) (justify left))
     )
-    (property "Footprint" "TestPoint:TestPoint_Pad_D2.0mm" (id 2) (at 144.78 71.12 0)
+    (property "Footprint" "TestPoint:TestPoint_Pad_D1.5mm" (id 2) (at 144.78 71.12 0)
       (effects (font (size 1.27 1.27)) hide)
     )
@@
       (effects (font (size 1.27 1.27)) (justify left))
     )
-    (property "Footprint" "TestPoint:TestPoint_Pad_D2.0mm" (id 2) (at 99.06 78.74 0)
+    (property "Footprint" "TestPoint:TestPoint_Pad_D1.5mm" (id 2) (at 99.06 78.74 0)
       (effects (font (size 1.27 1.27)) hide)
     )
@@
       (effects (font (size 1.27 1.27)) hide)
     )
+    (property "LCSC" "C17414" (id 5) (at 229.87 69.85 0)
+      (effects (font (size 1.27 1.27)) hide)
+    )
     (pin "1")
     (pin "2")
@@
       (effects (font (size 1.27 1.27)) hide)
     )
+    (property "LCSC" "C49678" (id 5) (at 118.364 62.738 0)
+      (effects (font (size 1.27 1.27)) hide)
+    )
     (pin "1")
     (pin "2")
@@
       (effects (font (size 1.27 1.27)) hide)
     )
+    (property "LCSC" "C17710" (id 5) (at 144.78 68.58 0)
+      (effects (font (size 1.27 1.27)) hide)
+    )
     (pin "1")
     (pin "2")
@@
       (effects (font (size 1.27 1.27)) (justify left))
     )
-    (property "Footprint" "TestPoint:TestPoint_Pad_D2.0mm" (id 2) (at 154.94 68.58 0)
+    (property "Footprint" "TestPoint:TestPoint_Pad_D1.5mm" (id 2) (at 154.94 68.58 0)
       (effects (font (size 1.27 1.27)) hide)
     )
@@
       (effects (font (size 1.27 1.27)) (justify left))
     )
-    (property "Footprint" "footprint:SOT-23-3_L2.9-W1.6-P1.90-LS2.8-BR" (id 2) (at 223.52 80.01 0)
+    (property "Footprint" "Package_TO_SOT_SMD:SOT-23-3" (id 2) (at 223.52 80.01 0)
       (effects (font (size 1.27 1.27) italic) hide)
     )
@@
       (effects (font (size 1.27 1.27)) hide)
     )
+    (property "LCSC" "C9002" (id 5) (at 85.09 109.22 0)
+      (effects (font (size 1.27 1.27)) hide)
+    )
     (pin "1")
     (pin "2")
@@
       (effects (font (size 1.27 1.27)) hide)
     )
+    (property "LCSC" "C17710" (id 5) (at 144.78 71.12 0)
+      (effects (font (size 1.27 1.27)) hide)
+    )
     (pin "1")
     (pin "2")
@@
       (effects (font (size 1.27 1.27)) hide)
     )
+    (property "LCSC" "C1804" (id 5) (at 93.98 113.03 0)
+      (effects (font (size 1.27 1.27)) hide)
+    )
     (pin "1")
     (pin "2")
@@
       (effects (font (size 1.27 1.27)) hide)
     )
+    (property "LCSC" "C1804" (id 5) (at 73.66 113.03 0)
+      (effects (font (size 1.27 1.27)) hide)
+    )
     (pin "1")
     (pin "2")
@@
       (effects (font (size 1.27 1.27)) (justify left))
     )
-    (property "Footprint" "TestPoint:TestPoint_Pad_D2.0mm" (id 2) (at 109.22 76.2 0)
+    (property "Footprint" "TestPoint:TestPoint_Pad_D1.5mm" (id 2) (at 109.22 76.2 0)
       (effects (font (size 1.27 1.27)) hide)
     )
@@
       (effects (font (size 1.27 1.27)) hide)
     )
+    (property "LCSC" "C17414" (id 5) (at 229.87 86.36 0)
+      (effects (font (size 1.27 1.27)) hide)
+    )
     (pin "1")
     (pin "2")
@@
       (effects (font (size 1.27 1.27)) hide)
     )
+    (property "LCSC" "C14267" (id 5) (at 129.54 78.74 0)
+      (effects (font (size 1.27 1.27)) hide)
+    )

Commit message: library changes, fixed model for dc jack
Other:
- title: IoT LED Strip Driver -> Spotify Reactive IoT LED Strip Driver
Changed lines of the file:
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@@
   (paper "A4")
   (title_block
-    (title "IoT LED Strip Driver")
+    (title "Spotify Reactive IoT LED Strip Driver")
     (date "2023-08-13")
-    (rev "v1.0")
+    (rev "v1.8-a")
     (comment 1 "A modular, internet connected LED strip driver")
+    (comment 2 "that reacts to the currently playing song on spotify")
   )
   (junction (at 236.22 69.85) (diameter 0) (color 0 0 0 0)
