File: iot_led_strip_pcb.kicad_pcb (KiCad board)
At the start: 2 copper layers, 80.9 x 70 mm, 7 parts

Commit message: did layout, whoops
Parts:
- added C1: 10uF, Capacitor_SMD:C_0805_2012Metric_Pad1.18x1.45mm_HandSolder, F.Cu at (153.0, 87.5)
- added C10: 22pF, Capacitor_SMD:C_0805_2012Metric_Pad1.18x1.45mm_HandSolder, F.Cu at (132.5, 102.2)
- added C11: 22pF, Capacitor_SMD:C_0805_2012Metric_Pad1.18x1.45mm_HandSolder, F.Cu at (132.5, 94.2)
- added C12: 100nF, Capacitor_SMD:C_0805_2012Metric_Pad1.18x1.45mm_HandSolder, F.Cu at (153.0, 89.8)
- added C13: 10uF, Capacitor_SMD:C_0805_2012Metric_Pad1.18x1.45mm_HandSolder, F.Cu at (153.0, 92.0)
- added C2: 10uF, Capacitor_SMD:C_0805_2012Metric_Pad1.18x1.45mm_HandSolder, F.Cu at (144.8, 81.0)
- added C3: 10uF, Capacitor_SMD:C_0805_2012Metric_Pad1.18x1.45mm_HandSolder, F.Cu at (142.3, 81.0)
- added C4: 100nF, Capacitor_SMD:C_0805_2012Metric_Pad1.18x1.45mm_HandSolder, F.Cu at (149.6, 81.0)
- added C5: 10uF, Capacitor_SMD:C_0805_2012Metric_Pad1.18x1.45mm_HandSolder, F.Cu at (151.8, 81.0)
- added C6: 100nF, Capacitor_SMD:C_0805_2012Metric_Pad1.18x1.45mm_HandSolder, F.Cu at (147.3, 81.0)
- added C7: 10uF, Capacitor_SMD:C_0805_2012Metric_Pad1.18x1.45mm_HandSolder, F.Cu at (130.5, 109.3)
- added C8: 47pF, Capacitor_SMD:C_0805_2012Metric_Pad1.18x1.45mm_HandSolder, F.Cu at (122.9, 104.2)
- added C9: 47pF, Capacitor_SMD:C_0805_2012Metric_Pad1.18x1.45mm_HandSolder, F.Cu at (122.9, 109.0)
- added D1: SMF5V0A, Diode_SMD:D_SMF, F.Cu at (131.3, 77.4)
- added D2: SMF5V0A, Diode_SMD:D_SMF, F.Cu at (131.3, 80.2)
- added D3: 1N5819WS, Diode_SMD:D_SOD-323_HandSoldering, F.Cu at (142.3, 76.5)
- added D4: LED, LED_SMD:LED_0805_2012Metric_Pad1.15x1.40mm_HandSolder, F.Cu at (147.0, 86.0)
- added D5: PWR_LED, LED_SMD:LED_0805_2012Metric_Pad1.15x1.40mm_HandSolder, F.Cu at (149.4, 86.0)
- added J1: I2C Expansion, Connector_PinHeader_2.54mm:PinHeader_1x04_P2.54mm_Vertical, F.Cu at (112.8, 78.8)
- added J2: Conn_01x03_Socket, Connector_PinHeader_2.54mm:PinHeader_1x03_P2.54mm_Vertical, F.Cu at (134.2, 72.5)
- added J3: GT-USB-7010ASV, footprint:USB-C-SMD_G-SWITCH_GT-USB-7010ASV, F.Cu at (115.2, 107.2)
- added J4: Barrel_Jack_Switch_Pin3Ring, Connector_BarrelJack:BarrelJack_Wuerth_6941xx301002, F.Cu at (123.8, 95.5)
- added J5: TC2050-IDC_Cortex-M, Connector:Tag-Connect_TC2050-IDC-FP_2x05_P1.27mm_Vertical, F.Cu at (147.2, 114.4)
- added J6: Conn_01x03_Socket_Solderwire, Connector_Wire:SolderWire-0.5sqmm_1x03_P4.6mm_D0.9mm_OD2.1mm_Relief, B.Cu at (119.5, 85.0)
- added JP1: SolderJumper_2_Open, Jumper:SolderJumper-2_P1.3mm_Open_RoundedPad1.0x1.5mm, F.Cu at (136.8, 94.6)
- added JP2: SolderJumper_2_Open, Jumper:SolderJumper-2_P1.3mm_Open_RoundedPad1.0x1.5mm, F.Cu at (127.6, 104.4)
- added JP3: USB PWR, Jumper:SolderJumper-2_P1.3mm_Open_RoundedPad1.0x1.5mm, F.Cu at (127.8, 99.2)
- added JP4: Jumper_2_Bridged, Connector_PinHeader_2.54mm:PinHeader_1x02_P2.54mm_Vertical, F.Cu at (128.0, 92.9)
- added JP5: SolderJumper_2_Open, Jumper:SolderJumper-2_P1.3mm_Open_RoundedPad1.0x1.5mm, F.Cu at (127.6, 108.8)
- added JP6: SolderJumper_2_Open, Jumper:SolderJumper-2_P1.3mm_Open_RoundedPad1.0x1.5mm, F.Cu at (136.8, 101.8)
- added JP7: JTAG-VTREF, Jumper:SolderJumper-2_P1.3mm_Open_RoundedPad1.0x1.5mm, F.Cu at (154.2, 111.6)
- added Q1: BSS138, Package_TO_SOT_SMD:SOT-23, F.Cu at (134.9, 89.5)
- added R1: 10k, Resistor_SMD:R_0805_2012Metric_Pad1.20x1.40mm_HandSolder, F.Cu at (138.1, 89.6)
- added R10: 27R, Resistor_SMD:R_0805_2012Metric_Pad1.20x1.40mm_HandSolder, F.Cu at (125.2, 109.0)
- added R11: 100, Resistor_SMD:R_0805_2012Metric_Pad1.20x1.40mm_HandSolder, F.Cu at (147.1, 90.1)
- added R12: 100, Resistor_SMD:R_0805_2012Metric_Pad1.20x1.40mm_HandSolder, F.Cu at (149.4, 90.1)
- added R2: 10k, Resistor_SMD:R_0805_2012Metric_Pad1.20x1.40mm_HandSolder, F.Cu at (131.8, 89.6)
- added R3: 27R, Resistor_SMD:R_0805_2012Metric_Pad1.20x1.40mm_HandSolder, F.Cu at (125.2, 104.2)
- added R4: 10k, Resistor_SMD:R_0805_2012Metric_Pad1.20x1.40mm_HandSolder, F.Cu at (135.0, 109.3)
- added R5: 10k, Resistor_SMD:R_0805_2012Metric_Pad1.20x1.40mm_HandSolder, F.Cu at (132.8, 109.3)
- added R6: 0R, Resistor_SMD:R_0805_2012Metric_Pad1.20x1.40mm_HandSolder, F.Cu at (137.2, 99.2)
- added R7: 0R, Resistor_SMD:R_0805_2012Metric_Pad1.20x1.40mm_HandSolder, F.Cu at (137.2, 97.0)
- added R8: 5.1k, Resistor_SMD:R_0805_2012Metric_Pad1.20x1.40mm_HandSolder, F.Cu at (120.8, 104.2)
- added R9: 5.1k, Resistor_SMD:R_0805_2012Metric_Pad1.20x1.40mm_HandSolder, F.Cu at (120.8, 109.0)
- added SW1: RESET, Button_Switch_SMD:SW_SPST_TL3342, F.Cu at (128.3, 115.8)
- added SW2: FLASH, Button_Switch_SMD:SW_SPST_TL3342, F.Cu at (137.4, 115.8)
- added TP1: 5V, TestPoint:TestPoint_Pad_D2.0mm, F.Cu at (132.7, 83.6)
- added TP2: 3.3V, TestPoint:TestPoint_Pad_D2.0mm, F.Cu at (153.5, 84.5)
- added TP3: GND, TestPoint:TestPoint_Pad_D2.0mm, F.Cu at (141.3, 86.4)
- added U1: AMS1117-3.3, Package_TO_SOT_SMD:SOT-223-3_TabPin2, F.Cu at (148.4, 75.1)
- added U2: ESP32-S2-MINI-1, PCM_Espressif:ESP32-S2-MINI-1, F.Cu at (147.3, 101.3)
- added Y1: Crystal_40Mhz, Crystal:Crystal_SMD_3225-4Pin_3.2x2.5mm_HandSoldering, F.Cu at (132.4, 98.3)
- H1, H2, H3, H4: footprint MountingHole:MountingHole_3.2mm_M3_Pad_Via -> MountingHole:MountingHole_2.2mm_M2_Pad_Via
- moved FID2 73.5 mm to (111.6, 113.6)
- moved FID3 54.8 mm to (158.4, 113.6)
- moved H2 29.0 mm to (156.0, 74.0)
- moved H4 29.0 mm to (156.0, 116.0)
- moved FID1 26.9 mm to (158.4, 76.4)
- moved H1 1.49 mm to (114.0, 74.0)
- moved H3 1.35 mm to (114.0, 116.0), turned to 90 degrees
- renumbered FID3 to FID1, FID1 to FID2, FID2 to FID3
Routing:
- net Earth: track 0.00 -> 135.9 mm, vias 0 -> 30
- net +3.3V: track 0.00 -> 128.8 mm, vias 0 -> 8
- net +5V: track 0.00 -> 69.7 mm
- net VBUS: track 0.00 -> 55.0 mm
- net /SDA: track 0.00 -> 46.8 mm, vias 0 -> 4
- net /~{RST}: track 0.00 -> 45.4 mm, vias 0 -> 2
- net /SCL: track 0.00 -> 44.9 mm, vias 0 -> 4
- net /BOOT: track 0.00 -> 36.7 mm, vias 0 -> 4
- net /D_{IN}: track 0.00 -> 30.1 mm, vias 0 -> 1
- net /LV_DIN: track 0.00 -> 18.9 mm, vias 0 -> 2
- net /USB_D+: track 0.00 -> 17.7 mm
- net /USB_D-: track 0.00 -> 16.8 mm
- net /DN: track 0.00 -> 14.4 mm
- net /DP: track 0.00 -> 13.6 mm
- net /X0_R: track 0.00 -> 13.3 mm
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Other:
- board size 80.9 x 70 mm -> 50 x 50 mm
- board text added: "3V3"
- board text added: "5V"
- board text added: "5V DC"
- board text added: "D_{in}"
- board text added: "GND"
- board text added: "I2C SSD1306"
- board text added: "LED STRIP"
- board text added: "SCL"
- board text added: "SDA"
- board text added: "USB"

Commit message: added photos of v2 prototype and updated readme
Parts:
- added G***: LOGO, LOGO, B.Cu at (134.3, 115.8)
- added REF**: KiCad-Logo2_5mm_SilkScreen, Symbol:KiCad-Logo2_5mm_SilkScreen, B.Cu at (123.6, 115.6)
Routing:
- net Earth: track 135.9 -> 146.6 mm
Other:
- board text added: "0xjmux & tsnl"
- board text added: "Spotify Neopixel Visualizer"
- board text added: "v2.0-a 09-2023"
